File: badge/badge.kicad_pcb (KiCad board)
At the start: 2 copper layers, 25 parts, among them J1 Conn_01x03_Pin, SW1 SW_Push

Commit message: Some work on routing
Parts:
- added C3: 0.1uF, Capacitor_THT:CP_Radial_Tantal_D5.5mm_P2.50mm, F.Cu at (56.5, 115.9)
- added C4: 0.1uF, Capacitor_THT:CP_Radial_Tantal_D5.5mm_P2.50mm, F.Cu at (62.5, 115.9)
- added C5: 0.1uF, Capacitor_THT:CP_Radial_Tantal_D5.5mm_P2.50mm, F.Cu at (59.5, 123.7)
- moved IC3 220.2 mm to (103.4, 114.1), turned to -90 degrees
- moved IC5 194.7 mm to (103.4, 95.8), turned to -90 degrees
- moved R2 191.7 mm to (77.8, 173.3), turned to 180 degrees
- moved IC2 182.8 mm to (55.0, 158.3), turned to 90 degrees
- moved SW1 169.9 mm to (96.8, 161.4)
- moved R3 160.5 mm to (103.8, 169.3), turned to 180 degrees
- moved C2 159.4 mm to (62.9, 167.3)
- moved C1 157.4 mm to (82.2, 172.5), turned to -90 degrees
- moved IC6 157.2 mm to (75.4, 140.0), turned to 90 degrees
- moved IC1 153.5 mm to (88.4, 161.5), turned to -90 degrees
- moved R1 123.9 mm to (77.1, 162.0), turned to 180 degrees
- moved IC7 0.40 mm to (70.4, 92.6)
- moved Y1 0.40 mm to (64.9, 110.3)
- moved Y2 0.40 mm to (57.3, 87.3)
- moved J1 0.40 mm to (106.8, 92.3)
Routing:
- net /RST: track 0.00 -> 155.3 mm
- net +5V: track 0.00 -> 122.4 mm
- net /CLK: track 0.00 -> 108.3 mm
- net /VIA_CS: track 0.00 -> 70.3 mm
- net /A6: track 0.00 -> 66.8 mm
- net /A2: track 0.00 -> 66.8 mm
- net /A4: track 0.00 -> 66.6 mm
- net /A7: track 0.00 -> 66.6 mm
- net /A5: track 0.00 -> 66.6 mm
- net /A3: track 0.00 -> 66.6 mm
- net /A1: track 0.00 -> 66.6 mm
- net /A0: track 0.00 -> 66.6 mm
- net /A11: track 0.00 -> 46.3 mm
- net /A10: track 0.00 -> 46.2 mm
- net /A8: track 0.00 -> 38.6 mm
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- added copper zone on F.Cu, net +5V
- added copper zone on B.Cu, net GND
Other:
- board outline added: 52.2 x 139.2 mm
- board text added: "AS6C62256"
- board text added: "AT28C256"
